File: PCB/main.kicad_pcb (KiCad board)
At the start: 2 copper layers, 103 x 22.5 mm, 17 parts, among them J1 USB_C_Receptacle, J2 RJ45, J3 USB_C_Receptacle, J4 USB_C_Receptacle, M1 Fan_PC_Chassis, M2 Fan_PC_Chassis, M3 Fan_PC_Chassis, M4 Fan_PC_Chassis, SW1 SW_DPDT_x2, U2 LAN9512i

Commit message: wee
Parts:
- removed R6: R, Resistor_SMD:R_0815_2038Metric
- moved U2 59.9 mm to (143.5, 82.5), turned to 90 degrees
Routing:
- net D-UP: track 129.2 -> 33.5 mm
- net D-DOWN1: track 148.4 -> 54.7 mm, vias 0 -> 1
- net D+UP: track 133.1 -> 46.3 mm, vias 1 -> 0
- net Net-(J4-CC2): track 50.4 -> 128.5 mm, vias 0 -> 2
- net gnd: track 143.4 -> 101.2 mm, vias 5 -> 2
- net VBUSUP: track 54.4 -> 94.2 mm
- net Net-(U2B-USBRBIAS): track 26.4 -> 52.8 mm, vias 0 -> 2
- net Net-(U2A-VDD33A-Pad10): track 22.4 -> 0.00 mm, vias 4 -> 0
- net Net-(J4-CC1): track 60.1 -> 39.9 mm, vias 4 -> 1
- net Net-(U2B-RXN): track 53.5 -> 34.1 mm, vias 0 -> 1
- net Net-(U2B-PRTCTL2): track 82.2 -> 99.2 mm, vias 1 -> 0
- net Net-(U2B-PRTCTL3): track 68.5 -> 52.1 mm
- net Net-(J3-CC2): track 47.6 -> 33.4 mm
- net unconnected-(J3-SHIELD-PadS1): track 12.2 -> 0.00 mm
- net unconnected-(J1-SHIELD-PadS1): track 12.2 -> 0.00 mm
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Other:
- board size 103 x 22.5 mm -> 76.5 x 37.5 mm
