File: PCB/main.kicad_sch (KiCad schematic)
At the start: 1 part, among them U1 Raspberry_Pi_Pico

Commit message: doin stuff
Parts:
- removed U1: Raspberry_Pi_Pico, ScottoKeebs_MCU:Raspberry_Pi_Pico, symbol ScottoKeebs:MCU_Raspberry_Pi_Pico
- added J1, J3, J4: USB_C_Receptacle, Connector_USB:USB_C_Receptacle_Amphenol_12401548E4-2A_CircularHoles, symbol Connector:USB_C_Receptacle
- added J2: RJ45, Connector_RJ:RJ45_Amphenol_54602-x08_Horizontal, symbol Connector:RJ45
- added M1, M2, M3, M4: Fan_PC_Chassis, Connector:FanPinHeader_1x03_P2.54mm_Vertical, symbol Motor:Fan_PC_Chassis
- added R1, R2, R3, R4, R5, R6, R7: R, Resistor_SMD:R_0815_2038Metric, symbol Device:R
- added SW1: SW_DPDT_x2, Button_Switch_THT:SW_CK_JS202011CQN_DPDT_Straight, symbol Switch:SW_DPDT_x2
- added U2: LAN9512i, Package_DFN_QFN:QFN-64-1EP_9x9mm_P0.5mm_EP7.3x7.3mm, symbol Interface_Ethernet:LAN9512i
Connections:
- new net: U2.10 (VDD33A), U2.49 (VDD33A), U2.5 (VDD33A), U2.51 (VDD33A), U2.54 (VDD33A), U2.57 (VDD33A), U2.64 (VDD33A)
- new net: U2.15 (VDD18CORE), U2.38 (VDD18CORE)
- new net: J3.A4 (VBUS), J3.A9 (VBUS), J3.B4 (VBUS), J3.B9 (VBUS), U2.14 (PRTCTL2)
- new net: J4.A4 (VBUS), J4.A9 (VBUS), J4.B4 (VBUS), J4.B9 (VBUS), U2.16 (PRTCTL3)
- new net: J2.3, U2.52 (RXP)
- new net: J2.6, U2.53 (RXN)
- new net: J2.1, U2.55 (TXP)
- new net: J2.2, U2.56 (TXN)
- new net: R5.2, U2.63 (USBRBIAS)
- new net: M1.2 (+), M2.2 (+), M3.2 (+), M4.2 (+), SW1.1 (A)
- new net: J3.B5 (CC2), R1.2
- new net: J4.A5 (CC1), R3.2
- new net: J3.A5 (CC1), R4.2
- new net: J4.B5 (CC2), R2.2
- new net D+DOWN1: J4.A6 (D+), J4.B6 (D+), U2.2 (USBDP2)
- new net D+DOWN2: J3.A6 (D+), J3.B6 (D+), U2.4 (USBDP3)
- new net D+UP: J1.A6 (D+), J1.B6 (D+), U2.59 (USBDP0)
- new net D-DOWN1: J4.A7 (D-), J4.B7 (D-), U2.1 (USBDM2)
- new net D-DOWN2: J3.A7 (D-), J3.B7 (D-), U2.3 (USBDM3)
- new net D-UP: J1.A7 (D-), J1.B7 (D-), U2.58 (USBDM0)
- new net VBUSUP: J1.A4 (VBUS), J1.A9 (VBUS), J1.B4 (VBUS), J1.B9 (VBUS), SW1.2 (B), SW1.3 (C), U2.11 (VBUS_DET), U2.19 (VDD33IO), U2.27 (VDD33IO), U2.33 (VDD33IO), U2.39 (VDD33IO), U2.46 (VDD33IO)
- new net gnd: J1.A1 (GND), J1.A12 (GND), J1.B1 (GND), J1.B12 (GND), J3.A1 (GND), J3.A12 (GND), J3.B1 (GND), J3.B12 (GND), J4.A1 (GND), J4.A12 (GND), J4.B1 (GND), J4.B12 (GND), M1.1 (-), M2.1 (-), M3.1 (-), M4.1 (-), R1.1, R2.1, R3.1, R4.1, R5.1, R6.1, R7.1, U2.65 (GND)

Commit message: fixing PCB
Connections:
- net gnd: now also J1.S1 (SHIELD), J3.S1 (SHIELD), J4.S1 (SHIELD)
- net at R6.2: now also J1.B5 (CC2)
- net at J1.A5 (CC1): now also R7.2
Changed lines of the file:
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@@
+	(wire
+		(pts
+			(xy 44.45 30.48) (xy 45.72 30.48)
+		)
+		(stroke
+			(width 0)
+			(type default)
+		)
+	)
 	(wire
 		(pts
@@
 		(pts
 			(xy 199.39 30.48) (xy 199.39 27.94)
+		)
+		(stroke
+			(width 0)
+			(type default)
+		)
+	)
+	(wire
+		(pts
+			(xy 44.45 33.02) (xy 45.72 33.02)
 		)
 		(stroke
@@
 		)
 	)
+	(global_label "gnd"
+		(shape input)
+		(at 265.43 90.17 90)
+		(fields_autoplaced yes)
+		(effects
+			(font
+				(size 1.27 1.27)
+			)
+			(justify left)
+		)
+		(property "Intersheetrefs" "${INTERSHEET_REFS}"
+			(at 265.43 83.7378 90)
+			(effects
+				(font
+					(size 1.27 1.27)
+				)
+				(justify left)
+				(hide yes)
+			)
+		)
+	)
 	(global_label "VBUSUP"
 		(shape input)
@@
 	(global_label "gnd"
 		(shape input)
+		(at 22.86 91.44 270)
+		(fields_autoplaced yes)
+		(effects
+			(font
+				(size 1.27 1.27)
+			)
+			(justify right)
+		)
+		(property "Intersheetrefs" "${INTERSHEET_REFS}"
+			(at 22.86 97.8722 90)
+			(effects
+				(font
+					(size 1.27 1.27)
+				)
+				(justify right)
+				(hide yes)
+			)
+		)
+	)
+	(global_label "gnd"
+		(shape input)
 		(at 113.03 124.46 180)
 		(fields_autoplaced yes)
@@
 				(hide yes)
 			)
+		)
+	)
+	(global_label "gnd"
+		(shape input)
+		(at 266.7 13.97 90)
+		(fields_autoplaced yes)
+		(effects
+			(font
+				(size 1.27 1.27)
+			)
+			(justify left)
+		)
+		(property "Intersheetrefs" "${INTERSHEET_REFS}"
+			(at 266.7 7.5378 90)
+			(effects
+				(font
+					(size 1.27 1.27)
+				)
+				(justify left)
+				(hide yes)
+			)

Commit message: fixing things
Parts:
- added Y2: KC2520Z, Oscillator:Oscillator_SMD_Kyocera_KC2520Z-4Pin_2.5x2.0mm, symbol Oscillator:KC2520Z
Connections:
- net VBUSUP: now also Y2.4 (VCC)
- net gnd: now also Y2.1 (INH), Y2.2 (GND)
- net at U2.61 (XI): now also Y2.3 (CLK)
Changed lines of the file:
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@@
+	(wire
+		(pts
+			(xy 102.87 87.63) (xy 107.95 87.63)
+		)
+		(stroke
+			(width 0)
+			(type default)
+		)
+	)
 	(wire
 		(pts
@@
 	(wire
 		(pts
-			(xy 196.85 119.38) (xy 222.25 119.38)
+			(xy 107.95 91.44) (xy 118.11 91.44)
 		)
 		(stroke
@@
 	(wire
 		(pts
-			(xy 151.13 160.02) (xy 184.15 160.02)
+			(xy 196.85 119.38) (xy 222.25 119.38)
 		)
 		(stroke
@@
 	(wire
 		(pts
-			(xy 199.39 35.56) (xy 199.39 44.45)
+			(xy 151.13 160.02) (xy 184.15 160.02)
 		)
 		(stroke
@@
 	(wire
 		(pts
-			(xy 151.13 114.3) (xy 201.93 114.3)
+			(xy 199.39 35.56) (xy 199.39 44.45)
 		)
 		(stroke
@@
 	(wire
 		(pts
-			(xy 184.15 57.15) (xy 205.74 57.15)
+			(xy 151.13 114.3) (xy 201.93 114.3)
 		)
 		(stroke
@@
 	(wire
 		(pts
-			(xy 227.33 57.15) (xy 210.82 57.15)
+			(xy 184.15 57.15) (xy 205.74 57.15)
 		)
 		(stroke
@@
 	(wire
 		(pts
-			(xy 234.95 148.59) (xy 234.95 151.13)
+			(xy 227.33 57.15) (xy 210.82 57.15)
 		)
 		(stroke
@@
 	(wire
 		(pts
-			(xy 180.34 157.48) (xy 180.34 130.81)
+			(xy 234.95 148.59) (xy 234.95 151.13)
 		)
 		(stroke
@@
 	(wire
 		(pts
-			(xy 199.39 30.48) (xy 199.39 27.94)
+			(xy 180.34 157.48) (xy 180.34 130.81)
 		)
 		(stroke
@@
 	(wire
 		(pts
-			(xy 44.45 33.02) (xy 45.72 33.02)
+			(xy 199.39 30.48) (xy 199.39 27.94)
 		)
 		(stroke
@@
 	(wire
 		(pts
-			(xy 213.36 27.94) (xy 213.36 33.02)
+			(xy 44.45 33.02) (xy 45.72 33.02)
 		)
 		(stroke
@@
 	(wire
 		(pts
-			(xy 151.13 157.48) (xy 180.34 157.48)
+			(xy 213.36 27.94) (xy 213.36 33.02)
 		)
 		(stroke
@@
 	(wire
 		(pts
-			(xy 177.8 149.86) (xy 177.8 125.73)
+			(xy 107.95 87.63) (xy 107.95 91.44)
 		)
 		(stroke
@@
 	(wire
 		(pts
-			(xy 184.15 160.02) (xy 184.15 138.43)
+			(xy 151.13 157.48) (xy 180.34 157.48)
 		)
 		(stroke
@@
 		)
 	)
+	(wire
+		(pts
+			(xy 177.8 149.86) (xy 177.8 125.73)
+		)
+		(stroke
+			(width 0)
+			(type default)
+		)
+	)
+	(wire
+		(pts
+			(xy 184.15 160.02) (xy 184.15 138.43)
+		)
+		(stroke
+			(width 0)
+			(type default)
+		)
+	)
+	(global_label "VBUSUP"
+		(shape input)
+		(at 92.71 80.01 90)
+		(fields_autoplaced yes)
+		(effects
+			(font
+				(size 1.27 1.27)
+			)
+			(justify left)
+		)
+		(property "Intersheetrefs" "${INTERSHEET_REFS}"
+			(at 92.71 69.5257 90)
+			(effects
+				(font
+					(size 1.27 1.27)
+				)
+				(justify left)
+				(hide yes)
+			)
+		)
+	)
 	(global_label "D+UP"
 		(shape input)
@@
 	(global_label "gnd"
 		(shape input)
+		(at 92.71 95.25 270)
+		(fields_autoplaced yes)
+		(effects
+			(font
+				(size 1.27 1.27)
+			)
+			(justify right)
+		)
+		(property "Intersheetrefs" "${INTERSHEET_REFS}"
+			(at 92.71 101.6822 90)
+			(effects
+				(font
+					(size 1.27 1.27)
+				)
+				(justify right)
+				(hide yes)
+			)
+		)
+	)
+	(global_label "gnd"
+		(shape input)
 		(at 113.03 124.46 180)
 		(fields_autoplaced yes)
@@
 		(property "Intersheetrefs" "${INTERSHEET_REFS}"
 			(at 112.2219 111.76 0)
+			(effects
+				(font
+					(size 1.27 1.27)
+				)
+				(justify right)
+				(hide yes)
+			)
+		)
+	)
+	(global_label "gnd"
+		(shape input)
+		(at 82.55 87.63 180)
+		(fields_autoplaced yes)
+		(effects
+			(font
+				(size 1.27 1.27)
+			)
+			(justify right)
+		)
+		(property "Intersheetrefs" "${INTERSHEET_REFS}"
+			(at 76.1178 87.63 0)
 			(effects
 				(font
@@
 					(unit 1)
 				)
+			)
+		)
+	)
+	(symbol
+		(lib_id "Oscillator:KC2520Z")
+		(at 92.71 87.63 0)
+		(unit 1)
+		(exclude_from_sim no)
+		(in_bom yes)
+		(on_board yes)
+		(dnp no)
+		(fields_autoplaced yes)
+		(property "Reference" "Y2"
+			(at 106.68 81.2098 0)
+			(effects
+				(font
+					(size 1.27 1.27)
+				)
+			)
+		)
+		(property "Value" "KC2520Z"
+			(at 106.68 83.7498 0)
+			(effects
+				(font
+					(size 1.27 1.27)
+				)
+			)
+		)
+		(property "Footprint" "Oscillator:Oscillator_SMD_Kyocera_KC2520Z-4Pin_2.5x2.0mm"
+			(at 96.52 83.82 0)
+			(effects
+				(font
+					(size 1.27 1.27)
+				)
+				(hide yes)
+			)
+		)
+		(property "Datasheet" "https://global.kyocera.com/prdct/electro/product/pdf/clock_z_xz_e.pdf"
+			(at 96.52 83.82 0)
+			(effects
+				(font
+					(size 1.27 1.27)
+				)
+				(hide yes)
+			)
+		)
+		(property "Description" "1.8432MHz ~ 125MHz Crystal Oscillator"
+			(at 92.71 87.63 0)
+			(effects
+				(font
+					(size 1.27 1.27)
+				)
+				(hide yes)
+			)
+		)
+		(pin "4"
+		)
+		(pin "1"
+		)
+		(pin "2"
+		)
+		(pin "3"
+		)
+		(instances
+			(project ""
+				(path "/a786fbae-561d-4e31-9f5c-b78d49a8da54"
+					(reference "Y2")
+					(unit 1)
+				)

Commit message: fixing lots of things
Parts:
- removed J2: RJ45, Connector_RJ:RJ45_Amphenol_54602-x08_Horizontal, symbol Connector:RJ45
- added C1: 0.1 pF, Capacitor_SMD:C_0201_0603Metric, symbol Device:C_US
- added C10, C3, C4, C9: 0.1, Capacitor_SMD:C_0201_0603Metric, symbol Device:C_US
- added C11: 4.7, Capacitor_SMD:C_0201_0603Metric, symbol Device:C_US
- added C2: 33 pF, Capacitor_SMD:C_0201_0603Metric, symbol Device:C_US
- added C5: 0.1 uF, Capacitor_SMD:C_0201_0603Metric, symbol Device:C_US
- added C6: 330, Capacitor_SMD:C_0201_0603Metric, symbol Device:C_US
- added C8: 1.0, Capacitor_SMD:C_0201_0603Metric, symbol Device:C_US
- added FB1: FerriteBead, Inductor_SMD:L_Ferrocore_DLG-0302, symbol Device:FerriteBead
- added J6: RJ45_Amphenol_RJMG1BD3B8K1ANR, Connector_RJ:RJ45_Amphenol_RJMG1BD3B8K1ANR, symbol Connector:RJ45_Amphenol_RJMG1BD3B8K1ANR
- added R10, R11, R12, R13, R14: 10, Resistor_SMD:R_0201_0603Metric, symbol ScottoKeebs:Placeholder_Resistor
- added R15: 330, Resistor_SMD:R_0201_0603Metric, symbol Device:R
- added R16: 0.1 uF, Resistor_SMD:R_0201_0603Metric, symbol Device:R
- added R17: 39.2 K, Resistor_SMD:R_0201_0603Metric, symbol ScottoKeebs:Placeholder_Resistor
- added R18: 61.9 K, Resistor_SMD:R_0201_0603Metric, symbol ScottoKeebs:Placeholder_Resistor
- added R8: 1.0 M, Resistor_SMD:R_0201_0603Metric, symbol ScottoKeebs:Placeholder_Resistor
- added R9: 12.4k, Resistor_SMD:R_0201_0603Metric, symbol ScottoKeebs:Placeholder_Resistor
- R1, R2, R3, R4: value R -> 5.1k; footprint Resistor_SMD:R_0815_2038Metric -> Resistor_SMD:R_0201_0603Metric
- R5: value R -> 12.0 k; footprint Resistor_SMD:R_0815_2038Metric -> Resistor_SMD:R_0201_0603Metric
- R6, R7: footprint Resistor_SMD:R_0815_2038Metric -> Resistor_SMD:R_0201_0603Metric
Connections:
- net VBUSUP: now also U2.40 (TEST3), C1.2, R17.1; no longer U2.11 (VBUS_DET), Y2.4 (VCC)
- net gnd: now also U2.34 (TEST2), C10.1, C11.1, C2.1, C3.1, C4.2, C5.1, C6.1, C8.2, C9.1, J6.R8, J6.SH, R15.2, R16.2, R18.1, R8.1, R9.1; no longer J3.S1 (SHIELD), J4.S1 (SHIELD), Y2.1 (INH), Y2.2 (GND)
- net VDD33A: now reaches U2.10 (VDD33A), U2.49 (VDD33A), U2.5 (VDD33A), U2.51 (VDD33A), U2.54 (VDD33A), U2.57 (VDD33A), U2.64 (VDD33A)
- net VDD33A: now also R10.2, R11.2, R12.2, R13.2, R14.2
- net at U2.15 (VDD18CORE), U2.38 (VDD18CORE): now also C10.2, C11.2, C9.2
- net at U2.48 (VDD18ETHPLL): now also C4.1, FB1.1
- net at U2.61 (XI), Y2.3 (CLK): now also R8.2
- net at U2.62 (VDD18USBPLL): now also C8.1, FB1.2
- net at U2.50 (EXRES): now also R9.2
- net at U2.52 (RXP): now also J6.R3 (RD+), R11.1
- net at U2.53 (RXN): now also J6.R6 (RD-), R10.1
- net at U2.55 (TXP): now also J6.R1 (TD+), R13.1
- net at U2.56 (TXN): now also J6.R2 (TD-), R12.1
- new net: R17.2, R18.2, U2.11 (VBUS_DET)
- new net: C6.2, J3.S1 (SHIELD), R16.1
- new net: C5.2, J4.S1 (SHIELD), R15.1
- new net: C1.1, Y2.4 (VCC)
- new net: C3.2, J6.R4 (TCT), J6.R5 (RCT), R14.1
- new net: C2.2, Y2.1 (INH), Y2.2 (GND)
Other:
- note added: "0.1 pF"
- note added: "0.1 uF"
- note added: "1.0 uF"
- note added: "1.0M"
- note added: "10 om 1%"
- note added: "12.0 K"
- note added: "12.4 K"
- note added: "33 pF"
- note added: "39.2 K"
- note added: "4.7 uF"
- note added: "5.1k"
- note added: "61.9 K"
- moved on the sheet: J3, R1, R4

Commit message: fixing things
Parts:
- added C7: 0.1 uF, Capacitor_SMD:C_0201_0603Metric, symbol Device:C_US
- added R19: 330, Resistor_SMD:R_0201_0603Metric, symbol Device:R
Connections:
- net gnd: now also C7.1, R19.2; no longer J1.S1 (SHIELD)
- new net: C7.2, J1.S1 (SHIELD), R19.1
Changed lines of the file:
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@@
 	)
 	(junction
+		(at 16.51 99.06)
+		(diameter 0)
+		(color 0 0 0 0)
+	)
+	(junction
 		(at 210.82 57.15)
 		(diameter 0)
@@
 	)
 	(junction
+		(at 16.51 91.44)
+		(diameter 0)
+		(color 0 0 0 0)
+	)
+	(junction
 		(at 166.37 147.32)
 		(diameter 0)
@@
 	)
 	(junction
+		(at 30.48 99.06)
+		(diameter 0)
+		(color 0 0 0 0)
+	)
+	(junction
 		(at 163.83 132.08)
 		(diameter 0)
@@
 	(wire
 		(pts
+			(xy 16.51 91.44) (xy 6.35 91.44)
+		)
+		(stroke
+			(width 0)
+			(type default)
+		)
+	)
+	(wire
+		(pts
 			(xy 210.82 60.96) (xy 213.36 60.96)
 		)
@@
 	(wire
 		(pts
+			(xy 30.48 100.33) (xy 30.48 99.06)
+		)
+		(stroke
+			(width 0)
+			(type default)
+		)
+	)
+	(wire
+		(pts
 			(xy 163.83 160.02) (xy 153.67 160.02)
 		)
@@
 	(wire
 		(pts
+			(xy 16.51 99.06) (xy 6.35 99.06)
+		)
+		(stroke
+			(width 0)
+			(type default)
+		)
+	)
+	(wire
+		(pts
 			(xy 163.83 144.78) (xy 151.13 144.78)
 		)
@@
 	(wire
 		(pts
+			(xy 16.51 99.06) (xy 30.48 99.06)
+		)
+		(stroke
+			(width 0)
+			(type default)
+		)
+	)
+	(wire
+		(pts
 			(xy 205.74 44.45) (xy 227.33 44.45)
 		)
@@
 	(wire
 		(pts
+			(xy 30.48 99.06) (xy 30.48 91.44)
+		)
+		(stroke
+			(width 0)
+			(type default)
+		)
+	)
+	(wire
+		(pts
 			(xy 234.95 148.59) (xy 234.95 151.13)
 		)
@@
 	(wire
 		(pts
+			(xy 22.86 91.44) (xy 16.51 91.44)
+		)
+		(stroke
+			(width 0)
+			(type default)
+		)
+	)
+	(wire
+		(pts
 			(xy 199.39 30.48) (xy 199.39 27.94)
 		)
@@
 		)
 	)
-	(global_label "gnd"
-		(shape input)
-		(at 30.48 91.44 270)
-		(fields_autoplaced yes)
-		(effects
-			(font
-				(size 1.27 1.27)
-			)
-			(justify right)
-		)
-		(property "Intersheetrefs" "${INTERSHEET_REFS}"
-			(at 30.48 97.8722 90)
-			(effects
-				(font
-					(size 1.27 1.27)
-				)
-				(justify right)
-				(hide yes)
-			)
-		)
-	)
 	(global_label "VBUSUP"
 		(shape output)
@@
 	(global_label "gnd"
 		(shape input)
-		(at 22.86 91.44 270)
+		(at 83.82 104.14 270)
 		(fields_autoplaced yes)
 		(effects
@@
 		)
 		(property "Intersheetrefs" "${INTERSHEET_REFS}"
-			(at 22.86 97.8722 90)
+			(at 83.82 110.5722 90)
 			(effects
 				(font
@@
 	(global_label "gnd"
 		(shape input)
-		(at 83.82 104.14 270)
+		(at 113.03 124.46 180)
 		(fields_autoplaced yes)
 		(effects
@@
 		)
 		(property "Intersheetrefs" "${INTERSHEET_REFS}"
-			(at 83.82 110.5722 90)
+			(at 106.5978 124.46 0)
 			(effects
 				(font
@@
 	(global_label "gnd"
 		(shape input)
-		(at 113.03 124.46 180)
+		(at 199.39 162.56 270)
 		(fields_autoplaced yes)
 		(effects
@@
 		)
 		(property "Intersheetrefs" "${INTERSHEET_REFS}"
-			(at 106.5978 124.46 0)
+			(at 199.39 168.9922 90)
 			(effects
 				(font
@@
 		)
 	)
-	(global_label "gnd"
+	(global_label "VDD33A"
 		(shape input)
-		(at 199.39 162.56 270)
+		(at 128.27 30.48 90)
 		(fields_autoplaced yes)
 		(effects
@@
 				(size 1.27 1.27)
 			)
-			(justify right)
+			(justify left)
 		)
 		(property "Intersheetrefs" "${INTERSHEET_REFS}"
-			(at 199.39 168.9922 90)
+			(at 128.27 20.3586 90)
 			(effects
 				(font
 					(size 1.27 1.27)
 				)
-				(justify right)
+				(justify left)
 				(hide yes)
 			)
 		)
 	)
-	(global_label "VDD33A"
+	(global_label "gnd"
 		(shape input)
-		(at 128.27 30.48 90)
+		(at 30.48 100.33 270)
 		(fields_autoplaced yes)
 		(effects
@@
 				(size 1.27 1.27)
 			)
-			(justify left)
+			(justify right)
 		)
 		(property "Intersheetrefs" "${INTERSHEET_REFS}"
-			(at 128.27 20.3586 90)
+			(at 30.48 106.7622 90)
 			(effects
 				(font
 					(size 1.27 1.27)
 				)
-				(justify left)
+				(justify right)
 				(hide yes)
 			)
@@
 	(symbol
 		(lib_id "Device:R")
+		(at 16.51 95.25 0)
+		(unit 1)
+		(exclude_from_sim no)
+		(in_bom yes)
+		(on_board yes)
+		(dnp no)
+		(fields_autoplaced yes)
+		(property "Reference" "R19"
+			(at 13.97 96.5201 0)
+			(effects
+				(font
+					(size 1.27 1.27)
+				)
+				(justify right)
+			)
+		)
+		(property "Value" "330"
+			(at 13.97 93.9801 0)
+			(effects
+				(font
+					(size 1.27 1.27)
+				)
+				(justify right)
+			)
+		)
+		(property "Footprint" "Resistor_SMD:R_0201_0603Metric"
+			(at 14.732 95.25 90)
+			(effects
+				(font
+					(size 1.27 1.27)
+				)
+				(hide yes)
+			)
+		)
+		(property "Datasheet" "~"
+			(at 16.51 95.25 0)
+			(effects
+				(font
+					(size 1.27 1.27)
+				)
+				(hide yes)
+			)
+		)
+		(property "Description" "Resistor"
+			(at 16.51 95.25 0)
+			(effects
+				(font
+					(size 1.27 1.27)
+				)
+				(hide yes)
+			)
+		)
+		(pin "1"
+		)
+		(pin "2"
+		)
+		(instances
+			(project "main"
+				(path "/a786fbae-561d-4e31-9f5c-b78d49a8da54"
+					(reference "R19")
+					(unit 1)
+				)
+			)
+		)
+	)
+	(symbol
+		(lib_id "Device:R")
 		(at 271.78 86.36 180)
 		(unit 1)
@@
 					(unit 1)
 				)
+			)
+		)
+	)
+	(symbol
+		(lib_id "Device:C_US")
+		(at 6.35 95.25 180)
+		(unit 1)
+		(exclude_from_sim no)
+		(in_bom yes)
+		(on_board yes)
+		(dnp no)
+		(fields_autoplaced yes)
+		(property "Reference" "C7"
+			(at 2.54 96.2661 0)
+			(effects
+				(font
+					(size 1.27 1.27)
+				)
+				(justify left)
+			)
+		)
+		(property "Value" "0.1 uF"
+			(at 2.54 93.7261 0)
+			(effects
+				(font
+					(size 1.27 1.27)
+				)
+				(justify left)
+			)
+		)
+		(property "Footprint" "Capacitor_SMD:C_0201_0603Metric"
+			(at 6.35 95.25 0)
+			(effects
+				(font
+					(size 1.27 1.27)
+				)
+				(hide yes)
+			)
+		)
+		(property "Datasheet" ""
+			(at 6.35 95.25 0)
+			(effects
+				(font
+					(size 1.27 1.27)
+				)
+				(hide yes)
+			)
+		)
+		(property "Description" "capacitor, US symbol"
+			(at 6.35 95.25 0)
+			(effects
+				(font
+					(size 1.27 1.27)
+				)
+				(hide yes)
+			)
+		)
+		(pin "1"
+		)
+		(pin "2"
+		)
+		(instances
+			(project "main"
+				(path "/a786fbae-561d-4e31-9f5c-b78d49a8da54"
+					(reference "C7")
+					(unit 1)
+				)

Commit message: fixing things
Parts:
- removed J1, J3, J4: USB_C_Receptacle, Connector_USB:USB_C_Receptacle_Amphenol_12401548E4-2A_CircularHoles, symbol Connector:USB_C_Receptacle
- added J1, J2, J4: USB_C_Receptacle, footprintsweeeeee:12401826_AMP, symbol MINE:USB_C_Receptacle
Connections:
- net D+DOWN1: now also J4.A6 (D+), J4.B6 (D+)
- net D+DOWN2: now also J2.A6 (D+), J2.B6 (D+)
- net D+UP: now also J1.A6 (D+), J1.B6 (D+)
- net D-DOWN1: now also J4.A7 (D-), J4.B7 (D-)
- net D-DOWN2: now also J2.A7 (D-), J2.B7 (D-)
- net D-UP: now also J1.A7 (D-), J1.B7 (D-)
- net VBUSUP: now also J1.A4 (VBUS), J1.A9 (VBUS), J1.B4 (VBUS), J1.B9 (VBUS)
- net gnd: now also J1.A1 (GND), J1.A12 (GND), J1.B1 (GND), J1.B12 (GND), J2.A1 (GND), J2.A12 (GND), J2.B1 (GND), J2.B12 (GND), J4.A1 (GND), J4.A12 (GND), J4.B1 (GND), J4.B12 (GND)
- net at U2.14 (PRTCTL2): now also J2.A4 (VBUS), J2.A9 (VBUS), J2.B4 (VBUS), J2.B9 (VBUS)
- net at U2.16 (PRTCTL3): now also J4.A4 (VBUS), J4.A9 (VBUS), J4.B4 (VBUS), J4.B9 (VBUS)
- net at C6.2, R16.1: now also J2.S1 (SHIELD), J2.S2 (SHIELD), J2.S3 (SHIELD), J2.S4 (SHIELD)
- net at R1.2: now also J2.B5 (CC2)
- net at R3.2: now also J4.A5 (CC1)
- net at R6.2: now also J1.B5 (CC2)
- net at R7.2: now also J1.A5 (CC1)
- net at C7.2, R19.1: now also J1.S1 (SHIELD), J1.S2 (SHIELD), J1.S3 (SHIELD), J1.S4 (SHIELD)
- net at C5.2, R15.1: now also J4.S1 (SHIELD), J4.S2 (SHIELD), J4.S3 (SHIELD), J4.S4 (SHIELD)
- net at R4.2: now also J2.A5 (CC1)
- net at R2.2: now also J4.B5 (CC2)
